Commit message: 增加双机读关节角控制

File: ur_description/urdf/uu_robot.urdf.xacro (robot description, xacro)
@@ -15,7 +15,7 @@
   <link name="uu_support">
     <visual>
-      <origin rpy="0 0 0" xyz=" 0 0 0"/>
+      <origin rpy="0 0 0" xyz=" 0 0 -0.05"/>
       <geometry>
-        <box size="2 4 0.1"/>
+        <box size="1 2 0.1"/>
       </geometry>
       <material name = "gray">
@@ -27,10 +27,10 @@
   <parent link="uu_support"/>
   <child link="right_base_link"/>
-  <origin xyz="0 -1 0.05" rpy="0 0 0"/>
+  <origin xyz="0 -0.5 0.0" rpy="0 0 0"/>
 </joint>
 <joint name="left_base_link-box" type="fixed">
   <parent link="uu_support"/>
   <child link="left_base_link"/>
-  <origin xyz="0 1  0.05" rpy="0 0 0"/>
+  <origin xyz="0 0.5 0.0" rpy="0 0 0"/>
 </joint>
 </robot>
